File: Eagle/ISS-Notify.sch (EAGLE design)
At the start: 56 parts, among them J3 PROTOSPACE2, SW1 9077-1, U1 ATMEGA32U4, U2 MCP7940N, U3 TPS63001, U4 MCP73811, U5 TLC5971, U6 TLC5971, X1 8 MHz, X2 32.768 kHz

Commit message: test pin placement on board
Parts:
- added TESTCLOCK, TESTDATA, TESTGND, TESTSCL, TESTSDC, TESTVBAT: TESTPIN, ISS-Notify:TESTPIN
Connections:
- net GND: now also TESTGND.TEST
- net LED_CLK: now also TESTCLOCK.TEST
- net LED_DATA: now also TESTDATA.TEST
- net SCL: now also TESTSCL.TEST
- net SDA: now also TESTSDC.TEST
- net VBAT: now also TESTVBAT.TEST
Changed lines of the file:
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@@
 <part name="U$5" library="ISS-Notify" deviceset="LOGO" device="" value="V0.3"/>
 <part name="C17" library="rcl_custom" deviceset="C-EU" device="0603-C-NOSILK" value="1 uF"/>
+<part name="TESTVBAT" library="ISS-Notify" deviceset="TESTPIN" device=""/>
+<part name="TESTSCL" library="ISS-Notify" deviceset="TESTPIN" device=""/>
+<part name="TESTSDC" library="ISS-Notify" deviceset="TESTPIN" device=""/>
+<part name="TESTDATA" library="ISS-Notify" deviceset="TESTPIN" device=""/>
+<part name="TESTCLOCK" library="ISS-Notify" deviceset="TESTPIN" device=""/>
+<part name="TESTGND" library="ISS-Notify" deviceset="TESTPIN" device=""/>
+<part name="GND23" library="supply1" deviceset="GND" device=""/>
 </parts>
 <sheets>
@@
 <instance part="U$5" gate="G$1" x="22.86" y="22.86"/>
 <instance part="C17" gate="CE" x="93.98" y="170.18"/>
+<instance part="TESTVBAT" gate="G$1" x="99.06" y="177.8"/>
+<instance part="TESTSCL" gate="G$1" x="327.66" y="172.72"/>
+<instance part="TESTSDC" gate="G$1" x="332.74" y="172.72"/>
+<instance part="TESTDATA" gate="G$1" x="48.26" y="73.66"/>
+<instance part="TESTCLOCK" gate="G$1" x="53.34" y="73.66"/>
+<instance part="TESTGND" gate="G$1" x="340.36" y="68.58"/>
+<instance part="GND23" gate="1" x="340.36" y="63.5"/>
 </instances>
 <busses>
@@
 <pinref part="GND3" gate="1" pin="GND"/>
 <wire x1="45.72" y1="144.78" x2="45.72" y2="165.1" width="0.1524" layer="91"/>
+</segment>
+<segment>
+<pinref part="GND23" gate="1" pin="GND"/>
+<pinref part="TESTGND" gate="G$1" pin="TEST"/>
+<wire x1="340.36" y1="66.04" x2="340.36" y2="68.58" width="0.1524" layer="91"/>
 </segment>
 </net>
@@
 <label x="210.82" y="167.64" size="1.778" layer="95"/>
 </segment>
+<segment>
+<pinref part="TESTSCL" gate="G$1" pin="TEST"/>
+<wire x1="304.8" y1="172.72" x2="327.66" y2="172.72" width="0.1524" layer="91"/>
+</segment>
 </net>
 <net name="SDA" class="0">
@@
 <label x="210.82" y="170.18" size="1.778" layer="95"/>
 <pinref part="U1" gate="ATMEGA" pin="INT1_SDA_PD1"/>
+</segment>
+<segment>
+<pinref part="TESTSDC" gate="G$1" pin="TEST"/>
+<wire x1="304.8" y1="170.18" x2="332.74" y2="170.18" width="0.1524" layer="91"/>
+<wire x1="332.74" y1="170.18" x2="332.74" y2="172.72" width="0.1524" layer="91"/>
 </segment>
 </net>
@@
 <label x="88.9" y="172.72" size="1.778" layer="95"/>
 <pinref part="C17" gate="CE" pin="1"/>
-<wire x1="93.98" y1="172.72" x2="104.14" y2="172.72" width="0.1524" layer="91"/>
+<wire x1="93.98" y1="172.72" x2="99.06" y2="172.72" width="0.1524" layer="91"/>
 <junction x="93.98" y="172.72"/>
+<pinref part="TESTVBAT" gate="G$1" pin="TEST"/>
+<wire x1="99.06" y1="172.72" x2="104.14" y2="172.72" width="0.1524" layer="91"/>
+<wire x1="99.06" y1="172.72" x2="99.06" y2="177.8" width="0.1524" layer="91"/>
+<junction x="99.06" y="172.72"/>
 </segment>
 </net>
@@
 <label x="208.28" y="213.36" size="1.778" layer="95"/>
 </segment>
+<segment>
+<pinref part="TESTDATA" gate="G$1" pin="TEST"/>
+<wire x1="68.58" y1="71.12" x2="48.26" y2="71.12" width="0.1524" layer="91"/>
+<wire x1="48.26" y1="71.12" x2="48.26" y2="73.66" width="0.1524" layer="91"/>
+</segment>
 </net>
 <net name="LED_CLK" class="0">
@@
 <label x="208.28" y="215.9" size="1.778" layer="95"/>
 </segment>
-</net>
+<segment>
+<pinref part="TESTCLOCK" gate="G$1" pin="TEST"/>
+<wire x1="68.58" y1="73.66" x2="53.34" y2="73.66" width="0.1524" layer="91"/>
+</segment>
+</net>

Commit message: incrament board version on screen
Parts:
- U$5: value V0.3 -> V0.4
Changed lines of the file:
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@@
 <part name="U$4" library="ISS-Notify" deviceset="_4-BARE_MOUNTING_HOLE" device="/.300"/>
 <part name="C16" library="rcl_custom" deviceset="C-EU" device="0603-C-NOSILK" value="100 pF"/>
-<part name="U$5" library="ISS-Notify" deviceset="LOGO" device="" value="V0.3"/>
+<part name="U$5" library="ISS-Notify" deviceset="LOGO" device="" value="V0.4"/>
 <part name="C17" library="rcl_custom" deviceset="C-EU" device="0603-C-NOSILK" value="1 uF"/>
 <part name="TESTVBAT" library="ISS-Notify" deviceset="TESTPIN" device=""/>

Commit message: fixed annoying bolt landing, moved a via or two
Parts:
- U$1, U$2, U$3, U$4: value _4-BARE_MOUNTING_HOLE/.300 -> _4-BARE_MOUNTING_HOLE/.250; device ISS-Notify:_4-BARE_MOUNTING_HOLE/.300 -> ISS-Notify:_4-BARE_MOUNTING_HOLE/.250
Changed lines of the file:
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@@
 <part name="FRAME1" library="frames" deviceset="A3L-LOC" device="" value="ISS Notify"/>
 <part name="RESET" library="ISS-Notify" deviceset="SWITCH" device=""/>
-<part name="U$1" library="ISS-Notify" deviceset="_4-BARE_MOUNTING_HOLE" device="/.300"/>
-<part name="U$2" library="ISS-Notify" deviceset="_4-BARE_MOUNTING_HOLE" device="/.300"/>
-<part name="U$3" library="ISS-Notify" deviceset="_4-BARE_MOUNTING_HOLE" device="/.300"/>
-<part name="U$4" library="ISS-Notify" deviceset="_4-BARE_MOUNTING_HOLE" device="/.300"/>
+<part name="U$1" library="ISS-Notify" deviceset="_4-BARE_MOUNTING_HOLE" device="/.250" value="_4-BARE_MOUNTING_HOLE/.250"/>
+<part name="U$2" library="ISS-Notify" deviceset="_4-BARE_MOUNTING_HOLE" device="/.250" value="_4-BARE_MOUNTING_HOLE/.250"/>
+<part name="U$3" library="ISS-Notify" deviceset="_4-BARE_MOUNTING_HOLE" device="/.250" value="_4-BARE_MOUNTING_HOLE/.250"/>
+<part name="U$4" library="ISS-Notify" deviceset="_4-BARE_MOUNTING_HOLE" device="/.250" value="_4-BARE_MOUNTING_HOLE/.250"/>
 <part name="C16" library="rcl_custom" deviceset="C-EU" device="0603-C-NOSILK" value="100 pF"/>
 <part name="U$5" library="ISS-Notify" deviceset="LOGO" device="" value="V0.4"/>

Commit message: Fixed L1 packages, changed USB header. Passes ERC, DRC, rats. Ship it.
Parts:
- removed USB: CON_USB-MICRO-6GND, ISS-Notify:CON_USB-MICRO-6GND
- added J1: ZX62D-B-5P8, con-hirose-microusb:ZX62D-B-5P8
Connections:
- net GND: now also J1.GND, J1.SHLD@1, J1.SHLD@2, J1.SHLD@3, J1.SHLD@4, U1.AREF; no longer USB.5
- net N$4: now also J1.D+; no longer USB.3
- net N$5: now also J1.D-; no longer USB.2
- net VUSB: now also J1.VCC; no longer USB.1

Commit message: Added fiducials per Screaming Circuits blog postw.
Parts:
- added U$10, U$11, U$6, U$7, U$8, U$9: FIDUCIAL, adafruit:FIDUCIAL
Other:
- note added: "Fiducials"
Changed lines of the file:
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@@
 <setting verticaltext="up"/>
 </settings>
-<grid distance="0.01" unitdist="inch" unit="inch" style="dots" multiple="1" display="yes" altdistance="0.01" altunitdist="inch" altunit="inch"/>
+<grid distance="0.1" unitdist="inch" unit="inch" style="dots" multiple="1" display="yes" altdistance="0.01" altunitdist="inch" altunit="inch"/>
 <layers>
 <layer number="1" name="Top" color="4" fill="1" visible="no" active="no"/>
@@
 <layer number="54" name="bGND_GNDA" color="7" fill="1" visible="no" active="no"/>
 <layer number="56" name="wert" color="7" fill="1" visible="no" active="no"/>
+<layer number="57" name="tCAD" color="7" fill="1" visible="no" active="no"/>
 <layer number="59" name="Invisible" color="7" fill="1" visible="no" active="no"/>
 <layer number="61" name="stand" color="7" fill="1" visible="no" active="no"/>
@@
 <layer number="132" name="bMask" color="7" fill="1" visible="yes" active="yes"/>
 <layer number="144" name="Drill_legend" color="7" fill="1" visible="yes" active="yes"/>
+<layer number="150" name="Notes" color="7" fill="1" visible="no" active="yes"/>
 <layer number="151" name="HeatSink" color="7" fill="1" visible="yes" active="yes"/>
 <layer number="152" name="_bDocu" color="7" fill="1" visible="yes" active="yes"/>
+<layer number="153" name="FabDoc1" color="6" fill="1" visible="no" active="no"/>
+<layer number="154" name="FabDoc2" color="2" fill="1" visible="no" active="no"/>
+<layer number="155" name="FabDoc3" color="7" fill="15" visible="no" active="no"/>
 <layer number="199" name="Contour" color="7" fill="1" visible="yes" active="yes"/>
 <layer number="200" name="200bmp" color="7" fill="1" visible="yes" active="yes"/>
@@
 <part name="J1" library="con-hirose-microusb" deviceset="ZX62D-B-5P8" device=""/>
 <part name="GND24" library="supply1" deviceset="GND" device=""/>
+<part name="U$6" library="adafruit" deviceset="FIDUCIAL" device=""/>
+<part name="U$7" library="adafruit" deviceset="FIDUCIAL" device=""/>
+<part name="U$8" library="adafruit" deviceset="FIDUCIAL" device=""/>
+<part name="U$9" library="adafruit" deviceset="FIDUCIAL" device=""/>
+<part name="U$10" library="adafruit" deviceset="FIDUCIAL" device=""/>
+<part name="U$11" library="adafruit" deviceset="FIDUCIAL" device=""/>
 </parts>
 <sheets>
@@
 <text x="106.68" y="91.44" size="3.81" layer="97">Color LEDs</text>
 <text x="325.12" y="132.08" size="3.81" layer="97">Breakout Header</text>
+<text x="17.78" y="71.12" size="1.778" layer="97">Fiducials</text>
 </plain>
 <instances>
@@
 <instance part="J1" gate="G$1" x="22.86" y="111.76"/>
 <instance part="GND24" gate="1" x="137.16" y="175.26"/>
+<instance part="U$6" gate="G$1" x="17.78" y="86.36"/>
+<instance part="U$7" gate="G$1" x="17.78" y="78.74"/>
+<instance part="U$8" gate="G$1" x="25.4" y="78.74"/>
+<instance part="U$9" gate="G$1" x="25.4" y="86.36"/>
+<instance part="U$10" gate="G$1" x="33.02" y="86.36"/>
+<instance part="U$11" gate="G$1" x="33.02" y="78.74"/>
 </instances>
 <busses>

Commit message: Add fiducials to board and library. Passes DRC, ERC, rats.
Parts:
- J1: value ZX62D-B-5P8 -> CON_USB-MICRO-ZX62D-B-5P8; device con-hirose-microusb:ZX62D-B-5P8 -> ISS-Notify:CON_USB-MICRO-ZX62D-B-5P8
- U$10, U$11, U$6, U$7, U$8, U$9: device adafruit:FIDUCIAL -> ISS-Notify:FIDUCIAL
Other:
- note added: "3.3V OUTPUT"
- moved on the sheet: J1
Changed lines of the file:
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@@
 <setting verticaltext="up"/>
 </settings>
-<grid distance="0.1" unitdist="inch" unit="inch" style="dots" multiple="1" display="yes" altdistance="0.01" altunitdist="inch" altunit="inch"/>
+<grid distance="0.01" unitdist="inch" unit="inch" style="dots" multiple="1" display="yes" altdistance="0.01" altunitdist="inch" altunit="inch"/>
 <layers>
 <layer number="1" name="Top" color="4" fill="1" visible="no" active="no"/>
@@
 <part name="TESTGND" library="ISS-Notify" deviceset="TESTPIN" device=""/>
 <part name="GND23" library="supply1" deviceset="GND" device=""/>
-<part name="J1" library="con-hirose-microusb" deviceset="ZX62D-B-5P8" device=""/>
+<part name="J1" library="ISS-Notify" deviceset="CON_USB-MICRO-ZX62D-B-5P8" device=""/>
 <part name="GND24" library="supply1" deviceset="GND" device=""/>
-<part name="U$6" library="adafruit" deviceset="FIDUCIAL" device=""/>
-<part name="U$7" library="adafruit" deviceset="FIDUCIAL" device=""/>
-<part name="U$8" library="adafruit" deviceset="FIDUCIAL" device=""/>
-<part name="U$9" library="adafruit" deviceset="FIDUCIAL" device=""/>
-<part name="U$10" library="adafruit" deviceset="FIDUCIAL" device=""/>
-<part name="U$11" library="adafruit" deviceset="FIDUCIAL" device=""/>
+<part name="U$6" library="ISS-Notify" deviceset="FIDUCIAL" device=""/>
+<part name="U$7" library="ISS-Notify" deviceset="FIDUCIAL" device=""/>
+<part name="U$8" library="ISS-Notify" deviceset="FIDUCIAL" device=""/>
+<part name="U$9" library="ISS-Notify" deviceset="FIDUCIAL" device=""/>
+<part name="U$10" library="ISS-Notify" deviceset="FIDUCIAL" device=""/>
+<part name="U$11" library="ISS-Notify" deviceset="FIDUCIAL" device=""/>
 </parts>
 <sheets>
@@
 <text x="325.12" y="132.08" size="3.81" layer="97">Breakout Header</text>
 <text x="17.78" y="71.12" size="1.778" layer="97">Fiducials</text>
+<text x="96.52" y="236.22" size="1.778" layer="97">3.3V OUTPUT</text>
 </plain>
 <instances>
@@
 </segment>
 <segment>
-<wire x1="33.02" y1="114.3" x2="35.56" y2="114.3" width="0.1524" layer="91"/>
+<wire x1="30.48" y1="114.3" x2="35.56" y2="114.3" width="0.1524" layer="91"/>
 <pinref part="GND2" gate="1" pin="GND"/>
 <wire x1="35.56" y1="114.3" x2="43.18" y2="114.3" width="0.1524" layer="91"/>
@@
 <pinref part="J1" gate="G$1" pin="GND"/>
 <pinref part="J1" gate="G$1" pin="SHLD@1"/>
-<wire x1="33.02" y1="109.22" x2="35.56" y2="109.22" width="0.1524" layer="91"/>
+<wire x1="30.48" y1="109.22" x2="35.56" y2="109.22" width="0.1524" layer="91"/>
 <wire x1="35.56" y1="109.22" x2="35.56" y2="114.3" width="0.1524" layer="91"/>
 <junction x="35.56" y="114.3"/>
 <pinref part="J1" gate="G$1" pin="SHLD@2"/>
-<wire x1="33.02" y1="106.68" x2="35.56" y2="106.68" width="0.1524" layer="91"/>
+<wire x1="30.48" y1="106.68" x2="35.56" y2="106.68" width="0.1524" layer="91"/>
 <wire x1="35.56" y1="106.68" x2="35.56" y2="109.22" width="0.1524" layer="91"/>
 <junction x="35.56" y="109.22"/>
 <pinref part="J1" gate="G$1" pin="SHLD@3"/>
-<wire x1="33.02" y1="104.14" x2="35.56" y2="104.14" width="0.1524" layer="91"/>
+<wire x1="30.48" y1="104.14" x2="35.56" y2="104.14" width="0.1524" layer="91"/>
 <wire x1="35.56" y1="104.14" x2="35.56" y2="106.68" width="0.1524" layer="91"/>
 <junction x="35.56" y="106.68"/>
 <pinref part="J1" gate="G$1" pin="SHLD@4"/>
-<wire x1="33.02" y1="101.6" x2="35.56" y2="101.6" width="0.1524" layer="91"/>
+<wire x1="30.48" y1="101.6" x2="35.56" y2="101.6" width="0.1524" layer="91"/>
 <wire x1="35.56" y1="101.6" x2="35.56" y2="104.14" width="0.1524" layer="91"/>
 <junction x="35.56" y="104.14"/>
@@
 <segment>
 <pinref part="R1" gate="R" pin="1"/>
-<wire x1="53.34" y1="119.38" x2="33.02" y2="119.38" width="0.1524" layer="91"/>
+<wire x1="53.34" y1="119.38" x2="30.48" y2="119.38" width="0.1524" layer="91"/>
 <pinref part="J1" gate="G$1" pin="D+"/>
 </segment>
@@
 <segment>
 <pinref part="R2" gate="R" pin="1"/>
-<wire x1="33.02" y1="121.92" x2="53.34" y2="121.92" width="0.1524" layer="91"/>
+<wire x1="30.48" y1="121.92" x2="53.34" y2="121.92" width="0.1524" layer="91"/>
 <pinref part="J1" gate="G$1" pin="D-"/>
 </segment>
@@
 <junction x="45.72" y="172.72"/>
 <pinref part="J1" gate="G$1" pin="VCC"/>
-<wire x1="33.02" y1="124.46" x2="38.1" y2="124.46" width="0.1524" layer="91"/>
+<wire x1="30.48" y1="124.46" x2="38.1" y2="124.46" width="0.1524" layer="91"/>
 <wire x1="38.1" y1="124.46" x2="38.1" y2="172.72" width="0.1524" layer="91"/>
 </segment>

Commit message: Changed resistor values for the LED according to datasheet
Parts:
- R7, R8: value 1 k -> 10 k
Changed lines of the file:
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@@
 <?xml version="1.0" encoding="utf-8"?>
 <!DOCTYPE eagle SYSTEM "eagle.dtd">
-<eagle version="6.4">
+<eagle version="7.1.0">
 <drawing>
 <settings>
@@
 <setting verticaltext="up"/>
 </settings>
-<grid distance="0.01" unitdist="inch" unit="inch" style="dots" multiple="1" display="yes" altdistance="0.01" altunitdist="inch" altunit="inch"/>
+<grid distance="0.1" unitdist="inch" unit="inch" style="lines" multiple="1" display="no" altdistance="0.01" altunitdist="inch" altunit="inch"/>
 <layers>
 <layer number="1" name="Top" color="4" fill="1" visible="no" active="no"/>
@@
 <part name="U5" library="ISS-Notify" deviceset="TLC5971" device=""/>
 <part name="U6" library="ISS-Notify" deviceset="TLC5971" device=""/>
-<part name="R7" library="rcl_custom" deviceset="R-US_" device="0603-C-NOSILK" value="1 k"/>
-<part name="R8" library="rcl_custom" deviceset="R-US_" device="0603-C-NOSILK" value="1 k"/>
+<part name="R7" library="rcl_custom" deviceset="R-US_" device="0603-C-NOSILK" value="10 k"/>
+<part name="R8" library="rcl_custom" deviceset="R-US_" device="0603-C-NOSILK" value="10 k"/>
 <part name="GND18" library="supply1" deviceset="GND" device=""/>
 <part name="GND19" library="supply1" deviceset="GND" device=""/>
